File: ClockingBoard_Hardware/ClockingBoard_Hardware.kicad_pcb (KiCad board)
At the start: 2 copper layers, 6 parts, among them U1 OKI, U2 TM4C129E_Launchpad

Commit message: Layout and step
Parts:
- added G***: LOGO, MRDT_Silkscreens:z_sig_Andrew_Van_Horn_Sig_15mm, F.Cu at (9.14, 35.1)
- added REF**: 4_40_Hole, MRDT_Drill_Holes:4_40_Hole, F.Cu at (7.62, 3.81)
- added REF**: 4_40_Hole, MRDT_Drill_Holes:4_40_Hole, F.Cu at (45.1, 32.9)
- added REF**: 4_40_Hole, MRDT_Drill_Holes:4_40_Hole, F.Cu at (49.9, 21.1)
- added REF**: 4_40_Hole, MRDT_Drill_Holes:4_40_Hole, F.Cu at (2.81, 15.6)
- Conn2: footprint MRDT_Connectors:MOLEX_SL_07_Horizontal -> MRDT_Connectors:MOLEX_SL_07_Vertical
- U2: footprint MRDT_Shields:TM4C129E_Launchpad_X9_THT_BOTTOM -> MRDT_Shields:TM4C129E_Launchpad_FULL_THT_BOTTOM
- moved U2 119.9 mm to (124.5, 0.00), turned to 180 degrees
- moved C1 111.5 mm to (69.8, 30.1), turned to 270 degrees
- moved Conn2 111.3 mm to (96.5, 15.2), turned to 90 degrees
- moved Conn1 108.2 mm to (79.8, 26.5), turned to 180 degrees
- moved C2 102.9 mm to (69.8, 38.5), turned to 90 degrees
- moved U1 94.9 mm to (68.6, 29.2), turned to 270 degrees
Connections:
- U2 pad +3V3: +3V3 -> Net-(U2-Pad+3V3)
Routing:
- net +3V3: track 0.00 -> 86.0 mm
- net Sync2: track 0.00 -> 42.0 mm
- net ICG: track 0.00 -> 30.0 mm
- net Sync1: track 0.00 -> 29.7 mm
- net M: track 0.00 -> 29.0 mm
- net SH: track 0.00 -> 22.4 mm
- net /+12V: track 0.00 -> 10.5 mm
- added copper zone on B.Cu, net GND
- added copper zone on F.Cu, net GND
Other:
- board outline added: 124.5 x 55.9 mm
- board text added: "+3V3"
- board text added: "3.3V"
- board text added: "CCD Clocking Board, Rev1 mars Rover Design team Missouri S&T, 2019 Andrew Van Horn"
- board text added: "GND"
- board text added: "ICG"
- board text added: "M"
- board text added: "S1"
- board text added: "S2"
- board text added: "SH"
