File: ClockingBoard_Hardware/ClockingBoard_Hardware.kicad_pcb (KiCad board)
At the start: 2 copper layers, 124.5 x 55.9 mm, 11 parts, among them U1 OKI, U2 TM4C129E_Launchpad

Commit message: fixed gerbs
Other:
- board text added: "CCD Clocking Board, Rev1 Mars Rover Design Team Missouri S&T, 2019 Andrew Van Horn"
- board text removed: "CCD Clocking Board, Rev1 mars Rover Design team Missouri S&T, 2019 Andrew Van Horn"
Changed lines of the file:
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@@
       (xy -6.395956 -0.780515) (xy -6.39578 -0.780671) (xy -6.278558 -0.884008) (xy -6.152213 -0.877709)) (layer F.SilkS) (width 0.01))
   )
-  (gr_text "CCD Clocking Board, Rev1\nmars Rover Design team\nMissouri S&T, 2019\nAndrew Van Horn" (at 1.778 27.178) (layer F.SilkS)
+  (gr_text "CCD Clocking Board, Rev1\nMars Rover Design Team\nMissouri S&T, 2019\nAndrew Van Horn" (at 1.778 27.178) (layer F.SilkS)
     (effects (font (size 1.5 1.5) (thickness 0.3)) (justify left))
   )
