File: ClockingBoard_Hardware/ClockingBoard_Hardware.sch (KiCad schematic (older format))
At the start: 6 parts, among them U1 OKI, U2 TM4C129E_Launchpad

Commit message: Layout and step
Parts:
- added unit 5 of U2
- Conn2: footprint MRDT_Connectors:MOLEX_SL_07_Horizontal -> MRDT_Connectors:MOLEX_SL_07_Vertical
- U2: footprint MRDT_Shields:TM4C129E_Launchpad_X9_THT_BOTTOM -> (none)
Connections:
- net +3V3: now also U2.+3V3' (A2_1); no longer U2.+3V3 (A1_1)
Changed lines of the file:
@@
 EESchema Schematic File Version 4
+LIBS:ClockingBoard_Hardware-cache
 EELAYER 26 0
 EELAYER END
@@
 F 0 "U2" H 3900 2500 60  0000 L CNN
 F 1 "TM4C129E_Launchpad" H 4201 3042 60  0001 L CNN
-F 2 "MRDT_Shields:TM4C129E_Launchpad_X9_THT_BOTTOM" H 3900 2550 60  0001 C CNN
+F 2 "" H 3900 2550 60  0001 C CNN
 F 3 "" H 3900 2550 60  0001 C CNN
 	1    3900 2550
@@
 F 0 "U2" H 4500 2500 60  0000 C CNN
 F 1 "TM4C129E_Launchpad" H 4432 3721 60  0000 C CNN
-F 2 "MRDT_Shields:TM4C129E_Launchpad_X9_THT_BOTTOM" H 4400 2550 60  0001 C CNN
+F 2 "" H 4400 2550 60  0001 C CNN
 F 3 "" H 4400 2550 60  0001 C CNN
 	2    4400 2550
@@
 F 0 "U2" H 5600 2500 60  0000 L CNN
 F 1 "TM4C129E_Launchpad" H 5905 3042 60  0001 L CNN
-F 2 "MRDT_Shields:TM4C129E_Launchpad_X9_THT_BOTTOM" H 5600 2550 60  0001 C CNN
+F 2 "" H 5600 2550 60  0001 C CNN
 F 3 "" H 5600 2550 60  0001 C CNN
 	3    5600 2550
@@
 F 0 "U2" H 6200 2500 60  0000 C CNN
 F 1 "TM4C129E_Launchpad" H 6132 3721 60  0001 C CNN
-F 2 "MRDT_Shields:TM4C129E_Launchpad_X9_THT_BOTTOM" H 6100 2550 60  0001 C CNN
+F 2 "" H 6100 2550 60  0001 C CNN
 F 3 "" H 6100 2550 60  0001 C CNN
 	4    6100 2550
@@
 F 0 "Conn2" H 9077 3208 60  0000 L CNN
 F 1 "Molex_SL_07" H 9077 3102 60  0000 L CNN
-F 2 "MRDT_Connectors:MOLEX_SL_07_Horizontal" H 8950 3000 60  0001 C CNN
+F 2 "MRDT_Connectors:MOLEX_SL_07_Vertical" H 8950 3000 60  0001 C CNN
 F 3 "" H 8950 3000 60  0001 C CNN
 	1    8950 2800
@@
 L power:+3V3 #PWR0105
 U 1 1 5C844B50
-P 3650 1550
-F 0 "#PWR0105" H 3650 1400 50  0001 C CNN
-F 1 "+3V3" H 3665 1723 50  0000 C CNN
-F 2 "" H 3650 1550 50  0001 C CNN
-F 3 "" H 3650 1550 50  0001 C CNN
-	1    3650 1550
-	1    0    0    -1
-$EndComp
-Wire Wire Line
-	3650 1550 3650 1600
-Wire Wire Line
-	3650 1600 3700 1600
+P 3650 2850
+F 0 "#PWR0105" H 3650 2700 50  0001 C CNN
+F 1 "+3V3" H 3665 3023 50  0000 C CNN
+F 2 "" H 3650 2850 50  0001 C CNN
+F 3 "" H 3650 2850 50  0001 C CNN
+	1    3650 2850
+	1    0    0    -1
+$EndComp
+Wire Wire Line
+	3650 2850 3650 2900
 $Comp
 L power:GND #PWR0106
@@
 Wire Wire Line
 	6400 1600 6400 1650
+$Comp
+L MRDT_Shields:TM4C129E_Launchpad U2
+U 5 1 5C86F005
+P 3900 3850
+F 0 "U2" H 4201 4448 60  0000 L CNN
+F 1 "TM4C129E_Launchpad" H 4201 4342 60  0000 L CNN
+F 2 "" H 3900 3850 60  0001 C CNN
+F 3 "" H 3900 3850 60  0001 C CNN
+	5    3900 3850
+	1    0    0    -1
+$EndComp
+Wire Wire Line
+	3700 2900 3650 2900
 $EndSCHEMATC
