File: CCDBoard_Hardware/_autosave-CCDBoard_Hardware.kicad_pcb (KiCad board)
At the start: 2 copper layers, 25 parts, among them U1 S11639-01, U2 LT1818, U3 74HC541

Commit message: Maybe a good start
Parts:
- moved C10 132.5 mm to (179.1, 74.4), turned to 90 degrees
- moved C7 120.9 mm to (164.3, 42.2), turned to 90 degrees
- moved R4 99.4 mm to (172.0, 36.6), turned to 270 degrees
- moved C1 98.5 mm to (131.3, 22.1)
- moved C8 97.1 mm to (176.3, 32.8), turned to 270 degrees
- moved C9 96.3 mm to (174.5, 74.3), turned to 90 degrees
- moved R3 85.6 mm to (172.2, 48.1), turned to 90 degrees
- moved C2 79.5 mm to (131.3, 26.4)
- moved R2 76.9 mm to (144.3, 52.7), turned to 90 degrees
- moved C5 66.5 mm to (149.4, 52.7), turned to 90 degrees
- moved C4 56.1 mm to (139.4, 74.4), turned to 90 degrees
- moved C6 39.2 mm to (160.0, 42.1)
- moved C3 27.3 mm to (144.0, 74.4)
- moved TP1 7.64 mm to (171.6, 29.2)
- moved Conn2 7.64 mm to (167.1, 22.6)
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