File: CCDBoard_Hardware/CCDBoard_Hardware.kicad_pcb (KiCad board)
At the start: 2 copper layers, 24 parts, among them U1 S11639-01, U2 LT1818, U3 74HC541

Commit message: not bad
Parts:
- added C7: 22 µF/25 V, Capacitor_SMD:C_0805_2012Metric_Pad1.15x1.40mm_HandSolder, F.Cu at (144.8, 79.8)
- moved R4 42.8 mm to (118.5, 87.6), turned to 180 degrees
- moved C8 42.0 mm to (118.5, 85.1), turned to 0 degrees
- moved U2 38.8 mm to (119.4, 92.8), turned to 270 degrees
- moved R1 35.4 mm to (134.2, 77.5), turned to 180 degrees
- moved C10 32.6 mm to (152.4, 79.8), turned to 270 degrees
- moved C9 32.2 mm to (157.5, 79.6), turned to 270 degrees
- moved C2 19.1 mm to (154.9, 79.6)
- moved TP2 18.2 mm to (111.8, 78.7)
- moved Conn2 18.0 mm to (106.7, 83.8), turned to 270 degrees
- moved C5 17.5 mm to (127.9, 94.0), turned to 0 degrees
- moved Conn1 16.7 mm to (106.7, 97.8), turned to 270 degrees
- moved C1 14.0 mm to (147.3, 79.8)
- moved TP5 13.3 mm to (111.8, 99.1)
- moved TP3 13.0 mm to (111.8, 83.8)
- moved R2 12.6 mm to (121.9, 81.7)
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Routing:
- net GND: track 65.2 -> 0.00 mm
- net Net-(R1-Pad1): track 3.81 -> 44.1 mm
- net Net-(R3-Pad1): track 3.59 -> 37.0 mm, vias 0 -> 2
- net CLK_IN: track 35.5 -> 3.40 mm
- net Trig: track 7.61 -> 30.6 mm
- net +5V: track 3.87 -> 26.3 mm, vias 0 -> 3
- net CLK: track 54.3 -> 32.1 mm, vias 2 -> 1
- net Net-(C5-Pad1): track 25.9 -> 3.96 mm, vias 2 -> 0
- net ST: track 49.8 -> 31.1 mm
- net Trig_OUT: track 32.0 -> 15.9 mm
- net ST_IN: track 30.4 -> 16.9 mm
- net Net-(R2-Pad2): track 3.08 -> 16.0 mm
- net EOS: track 41.5 -> 31.9 mm, vias 2 -> 1
- net Net-(R3-Pad2): track 14.0 -> 9.04 mm
- net Video: track 10.7 -> 15.6 mm
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- added copper zone on B.Cu, net +5V
- added copper zone on F.Cu, net GND
- removed copper zone on F.Cu, net +5V
- removed copper zone on B.Cu, net GND

Commit message: Finished
thank god
Parts:
- removed TP5: CLKTestPoint, TestPoint:TestPoint_THTPad_D2.5mm_Drill1.2mm
- added CLK: CLKTestPoint, TestPoint:TestPoint_THTPad_D2.5mm_Drill1.2mm, F.Cu at (111.8, 101.9)
- added REF**: 4_40_Hole, MRDT_Drill_Holes:4_40_Hole, F.Cu at (105.4, 110.5)
- added REF**: 4_40_Hole, MRDT_Drill_Holes:4_40_Hole, F.Cu at (161.3, 110.5)
- added REF**: 4_40_Hole, MRDT_Drill_Holes:4_40_Hole, F.Cu at (161.3, 80.0)
- moved C3 48.7 mm to (122.8, 111.0), turned to 0 degrees
- moved C4 43.3 mm to (118.9, 110.0), turned to 90 degrees
- moved C2 39.5 mm to (119.3, 96.5), turned to 0 degrees
- moved C6 35.9 mm to (126.6, 78.7), turned to 180 degrees
- moved C7 33.2 mm to (115.6, 95.5), turned to 90 degrees
- moved C9 32.5 mm to (149.0, 111.0), turned to 180 degrees
- moved C1 30.8 mm to (153.2, 110.0), turned to 90 degrees
- moved C10 25.9 mm to (126.5, 80.8), turned to 180 degrees
- moved EOS 5.68 mm to (116.8, 81.3), turned to 270 degrees
- moved Trig 2.54 mm to (111.8, 81.3), turned to 270 degrees
- moved PreAmpVid 2.29 mm to (152.1, 94.0)
- moved C8 1.70 mm to (117.0, 85.9)
- moved R4 1.70 mm to (117.0, 88.4)
- turned ST to 270 degrees
- turned Video to 270 degrees
- renumbered TP3 to EOS, TP4 to PreAmpVid, TP6 to ST, TP2 to Trig, TP1 to Video
Routing:
- net Net-(R1-Pad1): track 44.1 -> 36.7 mm, vias 0 -> 1
- net ST: track 31.1 -> 35.7 mm, vias 2 -> 1
- net CLK: track 32.1 -> 35.9 mm, vias 1 -> 3
- net EOS_OUT: track 17.9 -> 14.9 mm, vias 2 -> 0
- net EOS: track 31.9 -> 34.8 mm
- net Net-(R3-Pad2): track 9.04 -> 11.3 mm, vias 0 -> 1
- net Trig: track 30.6 -> 32.6 mm
- net Net-(R3-Pad1): track 37.0 -> 36.0 mm
- net +5V: track 26.3 -> 27.2 mm, vias 3 -> 2
- net Video: track 15.6 -> 16.3 mm
- net Net-(R2-Pad2): vias 0 -> 2
Other:
- board outline added: 63.5 x 38.1 mm
- board text added: "5v"
- board text added: "CLK"
- board text added: "Eos"
- board text added: "GND"
- board text added: "ST"
- board text added: "Trig"
- board text added: "Vid"

Commit message: added silk screens
Parts:
- added G***: LOGO, MRDT_Silkscreens:masonsig, F.Cu at (158.1, 96.5)
- added G***: LOGO, MRDT_Silkscreens:sigsymsmoler, B.Cu at (161.0, 102.9)
Other:
- board text added: "CCD, REV. 1 MARS ROVER DESIGN TEAM MISSOURI S&T, 2020 Mason Akers"
