File: CCDBoard_Hardware/CCDBoard_Hardware.sch (KiCad schematic (older format))
At the start: 25 parts, among them U1 S11639-01, U2 LT1818, U3 74HC541

Commit message: same as the last. please dont be broken
Parts:
- removed C1, C10, C4, C7: 22 µF/25 V, Capacitor_SMD:C_0805_2012Metric_Pad1.15x1.40mm_HandSolder, symbol Device:CP_Small
- removed C2, C3, C6, C9: 0.1 µF, Capacitor_SMD:C_0603_1608Metric_Pad1.05x0.95mm_HandSolder, symbol Device:C_Small
- removed C5: 1 µF, Capacitor_SMD:C_0603_1608Metric_Pad1.05x0.95mm_HandSolder, symbol Device:C_Small
- removed C8: 22 pF, Capacitor_SMD:C_0603_1608Metric_Pad1.05x0.95mm_HandSolder, symbol Device:C_Small
- removed Conn1: Molex_SL_04 IN, MRDT_Connectors:MOLEX_SL_04_Vertical, symbol MRDT_Connectors:Molex_SL_04
- removed Conn2: Molex_SL_04 OUT, MRDT_Connectors:MOLEX_SL_04_Vertical, symbol MRDT_Connectors:Molex_SL_04
- removed R1, R2: 82 Ω, Resistor_SMD:R_0603_1608Metric_Pad1.05x0.95mm_HandSolder, symbol Device:R
- removed R3: 100 Ω, Resistor_SMD:R_0603_1608Metric_Pad1.05x0.95mm_HandSolder, symbol Device:R
- removed R4: 51 Ω, Resistor_SMD:R_0603_1608Metric_Pad1.05x0.95mm_HandSolder, symbol Device:R
- removed TP1: VideoTestPoint, TestPoint:TestPoint_THTPad_D2.5mm_Drill1.2mm, symbol Connector:TestPoint
- removed TP2: TrigTestPoint, TestPoint:TestPoint_THTPad_D2.5mm_Drill1.2mm, symbol Connector:TestPoint
- removed TP3: EOSTestPoint, TestPoint:TestPoint_THTPad_D2.5mm_Drill1.2mm, symbol Connector:TestPoint
- removed TP4: VideoPreAmpTestPoint, TestPoint:TestPoint_THTPad_D2.5mm_Drill1.2mm, symbol Connector:TestPoint
- removed TP5: CLKTestPoint, TestPoint:TestPoint_THTPad_D2.5mm_Drill1.2mm, symbol Connector:TestPoint
- removed TP6: STTestPoint, TestPoint:TestPoint_THTPad_D2.5mm_Drill1.2mm, symbol Connector:TestPoint
- removed U1: S11639-01, MRDT_Devices:CCD-S11639-01, symbol CCDBoard_Hardware-rescue:S11639-01-MRDT_ICs
- removed U2: LT1818, Package_TO_SOT_SMD:SOT-23-5_HandSoldering, symbol pspice:OPAMP
- removed U3: 74HC541, Package_SO:SOIC-20W_7.5x12.8mm_P1.27mm, symbol MRDT_ICs:74HC541
Connections:
- no-connect marks 24 -> 0
